File: STM32-FC/STM32-FC.kicad_pcb (KiCad board)
At the start: 4 copper layers, 39 x 48.5 mm, 129 parts, among them J1 GH 1.25mm 6P, J10 GH 1.25mm 10P, J11 GH 1.25mm 6P, J12 GH 1.25mm 6P, J13 GH 1.25mm 6P, J14 GH 1.25mm 4P, J15 GH 1.25mm 4P, J16 GH 1.25mm 4P, J2 USB_C_USB2.0_14P, J3 GH 1.25mm 6P, J4 TF-06A, J5 JST ZH 1.5mm 2P, J6 PWM_Conn_3x14, J7 ZH 1.5mm 4P, J8 GH 1.25mm 4P, J9 ZH 1.5mm 3P, Q1 PMDPB30XN, Q2 PMDPB30XN, Q3 PMDPB55XP, U1 STM32F407VETx, U10 LPS22HH, U11 TMUX1104, U12 ATA6561-GBQW, U13 ATA6561-GBQW, U2 USBLC6-2SC6, U3 TPS62840, U5 TPS62840, U6 W25X40CLUXIG, U7 BMI323, U8 ICM-42688-P, U9 LIS2MDLTR, Y1 16MHz

Commit message: stm32f103 add
Parts:
- added R38: 10k, Resistor_SMD:R_0402_1005Metric, F.Cu at (123.3, 52.1)
- added R39: 10k, Resistor_SMD:R_0402_1005Metric, F.Cu at (123.3, 54.1)
- added R40: 10k, Resistor_SMD:R_0402_1005Metric, F.Cu at (123.3, 56.1)
- added R41: 10k, Resistor_SMD:R_0402_1005Metric, F.Cu at (123.3, 58.1)
- added R42: 10k, Resistor_SMD:R_0402_1005Metric, F.Cu at (123.3, 60.1)
- added R43: 10k, Resistor_SMD:R_0402_1005Metric, F.Cu at (123.3, 62.1)
- added U4: STM32F103C8Tx, Package_QFP:LQFP-48_7x7mm_P0.5mm, F.Cu at (174.7, 91.3)
- H1, H2, H3, H4: footprint Hole:MountingHole_2.2mm_M2 -> MountingHole:MountingHole_2.2mm_M2_ISO7380_Pad
- J6: moved to F.Cu
- U10: footprint LPS22HH:ST_HLGA-10_2x2mm_P0.5mm_LayoutBorder3x2y -> Package_LGA:ST_HLGA-10_2x2mm_P0.5mm_LayoutBorder3x2y
- U11: footprint TMUX1104:TMUX1104 -> Package_SON:USON-10_2.5x1.0mm_P0.5mm
- U6: footprint W25X40CLUX:USON_LUXIG TR_WIN-L -> W25X40CLUX:USON_LUXIG_TR_HandSolder
- U7: footprint BMI323:BMI323_L -> BMI323:BMI323
- moved H2 79.4 mm to (85.0, 115.0)
- moved C14 66.1 mm to (154.0, 42.0)
- moved C16 66.1 mm to (159.2, 42.0)
- moved C17 66.1 mm to (155.5, 43.5)
- moved C19 66.1 mm to (160.8, 43.5)
- moved L1 66.1 mm to (157.5, 42.5)
- moved L3 66.1 mm to (162.8, 42.5)
- moved R20 66.1 mm to (156.0, 39.8)
- moved R22 66.1 mm to (161.2, 39.8)
- moved U3 66.1 mm to (155.5, 41.5)
- moved U5 66.1 mm to (160.8, 41.5)
- moved J6 59.5 mm to (94.6, 71.9), turned to 0 degrees
- moved Q2 50.2 mm to (178.7, 64.3)
- moved Q3 50.2 mm to (178.7, 66.8)
- moved R10 50.2 mm to (180.4, 64.3)
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Connections:
- J6 pad 1: /TIM4_CH2 -> unconnected-(J6-CH1-Pad1)
- J6 pad 10: /TIM3_CH4 -> unconnected-(J6-CH10-Pad10)
- J6 pad 11: /TIM1_CH2 -> unconnected-(J6-CH11-Pad11)
- J6 pad 12: /TIM1_CH3 -> unconnected-(J6-CH12-Pad12)
- J6 pad 13: /RSSI_IN -> unconnected-(J6-RSSI-Pad13)
- J6 pad 14: /RC_INPUT/RCIN -> /IO Processer/RCIN
- J6 pad 2: /TIM3_CH1 -> unconnected-(J6-CH2-Pad2)
- J6 pad 3: /TIM3_CH2 -> unconnected-(J6-CH3-Pad3)
- J6 pad 4: /TIM4_CH4 -> unconnected-(J6-CH4-Pad4)
- J6 pad 5: /TIM5_CH1 -> unconnected-(J6-CH5-Pad5)
- J6 pad 6: /TIM5_CH2 -> unconnected-(J6-CH6-Pad6)
- J6 pad 7: /TIM5_CH3 -> unconnected-(J6-CH7-Pad7)
- J6 pad 8: /TIM5_CH4 -> unconnected-(J6-CH8-Pad8)
- J6 pad 9: /TIM3_CH3 -> unconnected-(J6-CH9-Pad9)
- U1 pad 66: /I2C3_SDA -> /GPS1_SDA
- U1 pad 67: /I2C3_SCL -> /GPS1_SCL
- U1 pad 78: /UART4_TX -> /GPS1_TX
- U1 pad 79: /UART4_RX -> /GPS1_RX
- U2 pad 1: /USB & POWER/USB_CONN_D- -> unconnected-(U2-I/O1-Pad1)
- U2 pad 2: GND -> unconnected-(U2-GND-Pad2)
- U2 pad 3: /USB & POWER/USB_CONN_D+ -> unconnected-(U2-I/O2-Pad3)
- U2 pad 4: /USB_D+ -> unconnected-(U2-I/O2-Pad4)
- U2 pad 5: VBUS -> unconnected-(U2-VBUS-Pad5)
- U2 pad 6: /USB_D- -> unconnected-(U2-I/O1-Pad6)
- U7 pad 1: /SPI3_MISO -> /SPI1_MISO
- U7 pad 13: /SPI3_SCK -> /SPI1_SCK
- U7 pad 14: /SPI3_MOSI -> /SPI1_MOSI
- U9 pad 1: /SPI3_SCK -> /SPI1_SCK
- U9 pad 4: /SPI3_MOSI -> /SPI1_MOSI
- U9 pad 7: /SPI3_MISO -> /SPI1_MISO
