File: STM32-FC/STM32-FC.kicad_sch (KiCad schematic)
At the start: 35 parts, among them J1 GH 1.25mm 6P, Q1 PMDPB30XN, U1 STM32F407VETx, Y1 16MHz

Commit message: stm32f103 add
Parts:
- H1, H2, H3, H4: footprint Hole:MountingHole_2.2mm_M2 -> MountingHole:MountingHole_2.2mm_M2_ISO7380_Pad
Connections:
- net BARO_INT: no longer names the net of U1.38 (PE7)
- net GYRO1_INT: no longer names the net of U1.39 (PE8)
- net GYRO2_INT: no longer names the net of U1.8 (PC14)
- net I2C3_SCL renamed GPS1_SCL
- net I2C3_SDA renamed GPS1_SDA
- net TIM1_CH2: no longer names the net of U1.42 (PE11)
- net TIM1_CH3: no longer names the net of U1.44 (PE13)
- net TIM3_CH1: no longer names the net of U1.63 (PC6)
- net TIM3_CH2: no longer names the net of U1.64 (PC7)
- net TIM3_CH3: no longer names the net of U1.35 (PB0)
- net TIM3_CH4: no longer names the net of U1.36 (PB1)
- net TIM4_CH2: no longer names the net of U1.93 (PB7)
- net TIM4_CH4: no longer names the net of U1.62 (PD15)
- net TIM5_CH1: no longer names the net of U1.23 (PA0)
- net TIM5_CH2: no longer names the net of U1.24 (PA1)
- net TIM5_CH3: no longer names the net of U1.25 (PA2)
- net TIM5_CH4: no longer names the net of U1.26 (PA3)
- net UART4_RX renamed GPS1_RX
- net UART4_TX renamed GPS1_TX
Other:
- removed sheet GPS
- removed sheet RC_INPUT
- added sheet IO Processor (./schematic/io_Processor.kicad_sch)
- sheet Communication: file io_communication.kicad_sch -> ./schematic/io_communication.kicad_sch
- sheet Communication ports: added GPS1_I2C_SCL, GPS1_I2C_SDA, GPS1_UART_RX, GPS1_UART_TX, GPS2_I2C_SCL, GPS2_I2C_SDA, GPS2_UART_RX, GPS2_UART_TX; removed none
- sheet Memory: file memory.kicad_sch -> ./schematic/memory.kicad_sch
- sheet Sensors: file sensors.kicad_sch -> ./schematic/sensors.kicad_sch
- sheet Sensors ports: added none; removed BARO_INT, GYRO1_INT, GYRO2_INT, SS2_SPI_MISO, SS2_SPI_MOSI, SS2_SPI_SCK
- sheet USB & POWER: file usb.kicad_sch -> ./schematic/usb.kicad_sch
- note removed: "VDDA"
- moved on the sheet: C12, C13, H1, H2, H3, H4

Commit message: v2.0.0 beta init
Parts:
- removed U1: STM32F407VETx, Package_QFP:LQFP-100_14x14mm_P0.5mm, symbol MCU_ST_STM32F4:STM32F407VETx
- added C50, C51, C52, C54, C56, C57, C58, C59, C60, C61, C62, C63, C64, C65, C66, C69: 100nF, Capacitor_SMD:C_0402_1005Metric, symbol Device:C_Small
- added C53, C55: 1uF, Capacitor_SMD:C_0402_1005Metric, symbol Device:C_Small
- added C67, C68: 10pF, Capacitor_SMD:C_0402_1005Metric, symbol Device:C_Small
- added IC1: STM32F746NGH6, BGA216C80P15X15_1300X1300X110, symbol STM32F746NGH6:STM32F746NGH6_1
- added R10: 120, Resistor_SMD:R_0402_1005Metric, symbol Device:R_Small_US
- added R12: 10k, Resistor_SMD:R_0402_1005Metric, symbol Device:R_Small_US
- added Y3: 16MHz, Crystal:Crystal_SMD_Abracon_ABM8G-4Pin_3.2x2.5mm, symbol Device:Crystal_GND24_Small
Connections:
- net +3.3V: now also C50.1, C51.1, C52.2, C53.2, C54.2, C55.2, C56.1, C57.1, C58.1, C59.1, C60.1, C61.1, C62.1, C63.1, C64.1, C65.1, C66.1, IC1.C1 (VBAT), IC1.E10 (VDD_4), IC1.E7 (VDD_1), IC1.E8 (VDD_2), IC1.E9 (VDD_3), IC1.F11 (VDD_7), IC1.F4 (VDD_5), IC1.F5 (VDD_6), IC1.G11 (VDDUSB), IC1.G5 (VDD_8), IC1.H11 (VDD_10), IC1.H5 (VDD_9), IC1.J11 (VDD_12), IC1.J5 (VDD_11), IC1.K11 (VDD_14), IC1.K5 (VDD_13), IC1.L10 (VDD_18), IC1.L7 (VDD_15), IC1.L8 (VDD_16), IC1.L9 (VDD_17), IC1.P1 (VREF+), IC1.R1 (VDDA)
- net BOOT0: now also R12.1
- net GND: now also C50.2, C51.2, C52.1, C53.1, C54.1, C55.1, C56.2, C57.2, C58.2, C59.2, C60.2, C61.2, C62.2, C63.2, C64.2, C65.2, C66.2, C67.1, C68.2, C69.2, IC1.F10 (VSS), IC1.F2 (VSS), IC1.F6 (VSS), IC1.F7 (VSS), IC1.F8 (VSS), IC1.F9 (VSS), IC1.G10 (VSS), IC1.G6 (VSS), IC1.H10 (VSS), IC1.H6 (VSS), IC1.J10 (VSS), IC1.J6 (VSS), IC1.K10 (VSS), IC1.K6 (VSS), IC1.K7 (VSS), IC1.K8 (VSS), IC1.K9 (VSS), IC1.L6 (VSS), IC1.M1 (VSSA), IC1.N1 (VREF-), R12.2, Y3.2, Y3.4
- net NRST: now also C69.1, IC1.J1 (NRST)
- net OSC_IN: now also C67.2, Y3.1
- net OSC_OUT: now also R10.2
- net VCAP1: no longer C6.2
- net VCAP2: no longer C7.1
- new net: C6.2, IC1.E11 (VCAP_2)
- new net: C68.1, R10.1, Y3.3
- new net: C7.1, IC1.L11 (VCAP_1)
Other:
- sheet Sensors renamed AHRS
- sheet AHRS: file ./schematic/sensors.kicad_sch -> schematic/AHRS.kicad_sch
- note removed: "VBAT and VDD"
- moved on the sheet: C15, C2, C6, C7

Commit message: add basic circuit stm32f7
Parts:
- removed BZ1: FUET-4020, FUET-4020:FUET-4020, symbol Device:Buzzer
- removed C1, C4: 10pF, Capacitor_SMD:C_0402_1005Metric, symbol Device:C_Small
- removed C12, C53, C55: 1uF, Capacitor_SMD:C_0402_1005Metric, symbol Device:C_Small
- removed C13, C15, C3, C5, C50, C51, C52, C54, C59, C60, C61, C62, C63, C64, C65, C66, C69, C8: 100nF, Capacitor_SMD:C_0402_1005Metric, symbol Device:C_Small
- removed C6, C7: 2.2uF, Capacitor_SMD:C_0402_1005Metric, symbol Device:C_Small
- removed D1: B5819W, Diode_SMD:D_SOD-323, symbol Device:D_Schottky_Small
- removed H1, H2, H3, H4: MountingHole, MountingHole:MountingHole_2.2mm_M2_ISO7380_Pad, symbol Mechanical:MountingHole
- removed unit 2 of IC1
- removed unit 3 of IC1
- removed Q1: PMDPB30XN, Nexperia_SOT1118:Nexperia_SOT1118, symbol Nexperia_PMD:PMDPB30XN
- removed R1, R12, R2, R5: 10k, Resistor_SMD:R_0402_1005Metric, symbol Device:R_Small_US
- removed R3, R4: 120, Resistor_SMD:R_0402_1005Metric, symbol Device:R_Small_US
- removed Y1: 16MHz, Crystal:Crystal_SMD_Abracon_ABM8G-4Pin_3.2x2.5mm, symbol Device:Crystal_GND24_Small
- J1: value GH 1.25mm 6P -> SM06B-GHS-TBT
Connections:
- net CAN1_RX: now also IC1.B12 (PD0)
- net CAN1_STBY: now also IC1.F1 (PC15)
- net CAN1_TX: now also IC1.C12 (PD1)
- net CAN2_RX: now also IC1.L13 (PB12)
- net CAN2_STBY: now also IC1.R14 (PB14)
- net CAN2_TX: now also IC1.K14 (PB13)
- net GPS1_RX: now also IC1.R13 (PB11)
- net GPS1_SCL: now also IC1.A7 (PB8)
- net GPS1_SDA: now also IC1.B4 (PB9)
- net GPS1_TX: now also IC1.P12 (PB10)
- net PM_CURRENT: now also IC1.M3 (PC1)
- net PM_VOLTAGE: now also IC1.M2 (PC0)
- net SWCLK: now also IC1.A14 (PA14)
- net SWDIO: now also IC1.A15 (PA13)
- net USB_D+: now also IC1.C15 (PA11)
- net USB_D-: now also IC1.B15 (PA12)
- net SD_CK: now reaches IC1.A12 (PC12)
- net MAIN2: now reaches IC1.A8 (PB5)
- net MAIN1: now reaches IC1.A9 (PB4)
- net SD_D3: now reaches IC1.B13 (PC11)
- net SD_D2: now reaches IC1.B14 (PC10)
- net SD_DET: now reaches IC1.D1 (PC13)
- net SD_CMD: now reaches IC1.D12 (PD2)
- net RC1_RX: now reaches IC1.D15 (PA10)
- net OSC_IN: no longer names the net of C67.2, Y3.1
- net OSC_IN: now also IC1.G1 (PH0)
- net OSC_OUT: no longer names the net of R10.2
- net OSC_OUT: now also IC1.H1 (PH1)
- new net AHRS1_MISO: IC1.P3 (PA6)
- new net AHRS1_MOSI: IC1.R3 (PA7)
- new net AHRS1_SCK: IC1.P4 (PA5)
- new net BARO1_NSS: IC1.F15 (PA8)
- new net GPS2_RX: IC1.N2 (PA1)
- new net GPS2_TX: IC1.N3 (PA0)
- new net IMU1_NSS: IC1.N4 (PA4)
- new net MAIN3: IC1.R5 (PB0)
- new net MAIN4: IC1.R4 (PB1)
- new net PWM_VOLTAGE: IC1.M4 (PC2)
- new net RC1_TX: IC1.E15 (PA9)
- new net RC2_RX: IC1.P2 (PA2)
- new net RC2_TX: IC1.R2 (PA3)
- new net SD_D0: IC1.G14 (PC8)
- new net SD_D1: IC1.F14 (PC9)
- new net TELEM2_CTS: IC1.L12 (PD14)
- new net TELEM2_RTS: IC1.K13 (PD15)
- new net VTX_VOLTAGE: IC1.L4 (PC3)
- no-connect marks 1 -> 7
Other:
- sheet Communication renamed IO
- removed sheet IO Processor
- added sheet STM32_io (schematic/STM32_io.kicad_sch)
- sheet AHRS ports: added none; removed BARO_NSS, GYRO1_NSS, GYRO2_NSS, MAG_NSS, SS_SPI_MISO, SS_SPI_MOSI, SS_SPI_SCK, V_BATT
- sheet IO ports: added none; removed CAN1_RX, CAN1_STBY, CAN1_TX, CAN2_RX, CAN2_STBY, CAN2_TX, GPS1_I2C_SCL, GPS1_I2C_SDA, GPS1_UART_RX, GPS1_UART_TX, GPS2_I2C_SCL, GPS2_I2C_SDA, GPS2_UART_RX, GPS2_UART_TX, I2C_SCL, I2C_SDA, UART2_CTS, UART2_RTS, UART2_RX, UART2_TX, UART3_CTS, UART3_RTS, UART3_RX, UART3_TX
- sheet Memory ports: added none; removed FLASH_NSS, MEM_SPI_MISO, MEM_SPI_MOSI, MEM_SPI_SCK, MSD_DETECT, MSD_NSS
- sheet USB & POWER ports: added none; removed PWR_SEL0, PWR_SEL1, USB_D+, USB_D-
- note added: "ADC123_IN10"
- note added: "ADC123_IN11"
- note added: "ADC123_IN12"
- note added: "ADC123_IN13"
- note added: "CAN1_RX"
- note added: "CAN1_TX"
- note added: "CAN2_RX"
- note added: "CAN2_TX"
- note added: "I2C1_SCL"
- note added: "I2C1_SDA"
- note added: "PA8"
- note added: "SPI1_MISO"
- note added: "SPI1_MOSI"
- note added: "SPI1_NSS"
- note added: "SPI1_SCK"
- note added: "TIM3_CH1"
- note added: "TIM3_CH2"
- note added: "TIM3_CH3"
- note added: "TIM3_CH4"
- note added: "UART1_RX"
- note added: "UART1_TX"
- note added: "UART2_RX"
- note added: "UART2_TX"
- note added: "UART4_RX"
- note added: "UART4_TX"
- note added: "USART3_RX"
- note added: "USART3_TX"
- note removed: "Buzzer"
- note removed: "Connectors"
- note removed: "M2"
- note removed: "Memory & SD Card"
- note removed: "Mounting Holes"
- note removed: "PD14 : TIM4_CH3"
- note removed: "Sensor Interface"
- moved on the sheet: C10, C11, C2, C56, C57, C58, C67, C68, C9, D2, D3, D4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

Commit message: add DJI Air unit and RC Selector
Parts:
- removed D2: Red, LED_SMD:LED_0402_1005Metric, symbol Device:LED_Small
- removed D3: Yellow, LED_SMD:LED_0402_1005Metric, symbol Device:LED_Small
- removed D4: Green, LED_SMD:LED_0402_1005Metric, symbol Device:LED_Small
- removed R6, R7, R8: 120, Resistor_SMD:R_0402_1005Metric, symbol Device:R_Small_US
Connections:
- net RC2_RX renamed VTX_RX
- net RC2_TX renamed VTX_TX
Other:
- note removed: "LEDs"
- note removed: "MCU"
- note removed: "W : PA4 R : PE0 Y : PE1 B : PE2"

Commit message: ERC passed
Parts:
- renumbered C2 to C1, C9 to C2, C10 to C3, C11 to C4, C56 to C5, C57 to C6, C58 to C7, C68 to C8, C67 to C9, R10 to R1, Y3 to Y1
Connections:
- no-connect marks 7 -> 22
Other:
- sheet USB & POWER ports: added none; removed PM_CURRENT, PM_VOLTAGE, SW_PWR_IMU
- note removed: "USB & POWER"
